Commit message: Fixed self-collisions in PyBullet but vamp still returning in collision for collision-free configurations in PyBullet.

File: resources/stretch/stretch_spherized.urdf (robot description, URDF)
Before this commit: robot stretch, 61 links, 60 joints
Links:
- added link link_theta
- added link link_y
- added link world
Joints:
- added joint joint_theta: type revolute, parent link_theta, child base_link, origin xyz=0 0 0 rpy=0 0 0, axis 0 0 1, limit lower=-3.14159 upper=3.14159 effort=100 velocity=1.0
- added joint joint_x: type prismatic, parent world, child link_y, origin xyz=0 0 0 rpy=0 0 0, axis 1 0 0, limit lower=-5.0 upper=5.0 effort=100 velocity=1.0
- added joint joint_y: type prismatic, parent link_y, child link_theta, origin xyz=0 0 0 rpy=0 0 0, axis 0 1 0, limit lower=-5.0 upper=5.0 effort=100 velocity=1.0
- joint joint_gripper_finger_left: origin xyz=0.0245029393015013 0 0.0371909405167127 rpy=-1.57079632679523 -1.48789318734672 -3.14159265358946 -> xyz=0.0245029393015013 0 0.0371909405167127 rpy=-1.57079632679523 -1.68789318734672 -3.14159265358946; type revolute -> fixed
- joint joint_gripper_finger_right: origin xyz=-0.0246929393014972 0 0.0371909405167257 rpy=-1.57079632679513 1.48789318732515 3.14159265358956 -> xyz=-0.0246929393014972 0 0.0371909405167257 rpy=-1.57079632679513 1.68789318732515 3.14159265358956; type revolute -> fixed

File: resources/stretch/stretch_spherized_sparse.urdf (robot description, URDF)
Before this commit: robot stretch, 61 links, 60 joints
Links:
- added link link_theta
- added link link_y
- added link world
Joints:
- added joint joint_theta: type revolute, parent link_theta, child base_link, origin xyz=0 0 0 rpy=0 0 0, axis 0 0 1, limit lower=-3.14159 upper=3.14159 effort=100 velocity=1.0
- added joint joint_x: type prismatic, parent world, child link_y, origin xyz=0 0 0 rpy=0 0 0, axis 1 0 0, limit lower=-5.0 upper=5.0 effort=100 velocity=1.0
- added joint joint_y: type prismatic, parent link_y, child link_theta, origin xyz=0 0 0 rpy=0 0 0, axis 0 1 0, limit lower=-5.0 upper=5.0 effort=100 velocity=1.0
- joint joint_gripper_finger_left: limit lower=0 upper=0 effort=0 velocity=0 -> lower=0 upper=0.3 effort=0 velocity=0; origin xyz=0.0245029393015013 0 0.0371909405167127 rpy=-1.57079632679523 -1.48789318734672 -3.14159265358946 -> xyz=0.0245029393015013 0 0.0371909405167127 rpy=-1.57079632679523 -1.68789318734672 -3.14159265358946; type revolute -> fixed
- joint joint_gripper_finger_right: limit lower=0 upper=0 effort=0 velocity=0 -> lower=0 upper=0.3 effort=0 velocity=0; origin xyz=-0.0246929393014972 0 0.0371909405167257 rpy=-1.57079632679513 1.48789318732515 3.14159265358956 -> xyz=-0.0246929393014972 0 0.0371909405167257 rpy=-1.57079632679513 1.68789318732515 3.14159265358956; type revolute -> fixed
